File: hardware/ecad/battery_sense.kicad_sch (KiCad schematic)
At the start: 0 parts

Commit message: finsihed 6/7 sheets, usb_data needs work. Some warnings to be dealt with aswell but no hard errors.
Parts:
- added C15: 100nF, Capacitor_SMD:C_01005_0402Metric, symbol Device:C
- added R11: 220k, Capacitor_SMD:C_0402_1005Metric, symbol Device:R
- added R12: 100k, Capacitor_SMD:C_0402_1005Metric, symbol Device:R
Connections:
- new net BAT: R12.2
- new net BAT_SENSE: C15.1, R11.2, R12.1
- new net GND: C15.2, R11.1
Other:
- company: (none) -> āvega systems
- title: (none) -> midi2BLE_Battery_Sense

Commit message: Updated schematics and added printed pdf
Parts:
- C15: footprint Capacitor_SMD:C_01005_0402Metric -> Capacitor_SMD:C_0402_1005Metric
Changed lines of the file:
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@@
 			)
 		)
-		(property "Footprint" "Capacitor_SMD:C_01005_0402Metric"
+		(property "Footprint" "Capacitor_SMD:C_0402_1005Metric"
 			(at 147.32 86.6648 0)
 			(hide yes)
